Commit message: Add physical adaptive gripper TCP frame

File: mycobot_ws/src/mycobot_description/urdf/mycobot_280_jn/mycobot_280_jn_adaptive_gripper.urdf (robot description, URDF)
Before this commit: robot mycobot_280_jn_adaptive_gripper, 14 links, 13 joints
Links:
- added link gripper_tcp
Joints:
- added joint gripper_base_to_tcp: type fixed, parent gripper_base, child gripper_tcp, origin xyz=0.0 0.0214 0.0003 rpy=0 0 0

Commit message: Add collision-aware arm model for physical planning

File: mycobot_ws/src/mycobot_description/urdf/mycobot_280_jn/mycobot_280_jn_adaptive_gripper.urdf (robot description, URDF)
Before this commit: robot mycobot_280_jn_adaptive_gripper, 15 links, 14 joints
Links:
- link joint1: geometry collision mesh filename=package://mycobot_description/urdf/mycobot_280_jn/collision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; visual mesh filename=package://mycobot_description/urdf/mycobot_280_jn/joint1_je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
- link joint2: geometry collision mesh filename=package://mycobot_description/urdf/mycobot_280_jn/collision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; visual mesh filename=package://mycobot_description/urdf/mycobot_280_jn/joint2.dae
- link joint3: geometry collision mesh filename=package://mycobot_description/urdf/mycobot_280_jn/collision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; visual mesh filename=package://mycobot_description/urdf/mycobot_280_jn/joint3.dae
- link joint4: geometry collision mesh filename=package://mycobot_description/urdf/mycobot_280_jn/collision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; visual mesh filename=package://mycobot_description/urdf/mycobot_280_jn/joint4.dae
- link joint5: geometry collision mesh filename=package://mycobot_description/urdf/mycobot_280_jn/collision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; visual mesh filename=package://mycobot_description/urdf/mycobot_280_jn/joint5.dae
- link joint6: geometry collision mesh filename=package://mycobot_description/urdf/mycobot_280_jn/collision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; visual mesh filename=package://mycobot_description/urdf/mycobot_280_jn/joint6.dae
- link joint6_flange: geometry collision mesh filename=package://mycobot_description/urdf/mycobot_280_jn/collision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; visual mesh filename=package://mycobot_description/urdf/mycobot_280_jn/joint7.dae
